Commit message: included link in urdf for transform required by slam_toolbox

File: resource/robot_webots.urdf (robot description, URDF)
Before this commit: robot robot, 11 links, 10 joints
Links:
- added link base_footprint
Joints:
- added joint base_footprint_joint: type fixed, parent base_link, child base_footprint, origin xyz=0 0 0 rpy=0 0 0

Commit message: adjusted robot dimensions and starting position

File: resource/robot_webots.urdf (robot description, URDF)
Before this commit: robot robot, 12 links, 11 joints
Links:
- link base_link: geometry collision cylinder length=1 radius=0.45; visual cylinder length=1 radius=0.45
Joints:
- joint base_link_camera_joint: origin xyz=0 0.4 0.9 rpy=-1.570796 0 0.009204 -> xyz=0 0.45 0.5 rpy=-1.570796 0 0.009204
- joint base_link_lidar_sensor_joint: origin xyz=0 0.4 1.15 rpy=0 0 1.57 -> xyz=0 0.4 0.55 rpy=0 0 1.57

Commit message: using new map, adjusted robot dimensions

File: resource/robot_webots.urdf (robot description, URDF)
Before this commit: robot C:/Users/guilh/Desktop/robot_webots.urdf, 12 links, 11 joints
Links:
- added link display
- added link obj_display
- link base_link: geometry collision cylinder length=0.5 radius=0.2; visual cylinder length=0.5 radius=0.2
- link motor_l1_solid: geometry collision cylinder length=0.1 radius=0.1; visual cylinder length=0.1 radius=0.1
- link motor_r1_solid: geometry collision cylinder length=0.1 radius=0.1; visual cylinder length=0.1 radius=0.1
Joints:
- added joint base_link_display_joint: type fixed, parent base_link, child display, origin xyz=0 0 0 rpy=0 0 0
- added joint base_link_obj_display_joint: type fixed, parent base_link, child obj_display, origin xyz=0 0 0 rpy=0 0 0
- joint base_link_camera_joint: origin xyz=0 0.45 0.5 rpy=-1.570796 0 0.009204 -> xyz=0 0.2 0.25 rpy=-1.570796 0 0.009204
- joint base_link_front support_joint: origin xyz=0 0.5 -0.477 rpy=0 0 0 -> xyz=0.002301 0.25 -0.499989 rpy=0 0 0
- joint base_link_lidar_sensor_joint: origin xyz=0 0.4 0.55 rpy=0 0 1.57 -> xyz=0 0.2 0.25 rpy=0 0 1.57
- joint base_link_rear support_joint: origin xyz=0 -0.5 -0.477 rpy=0 0 0 -> xyz=0 -0.25 -0.25 rpy=0 0 0
- joint motor_l1: origin xyz=-0.5 0 -0.35 rpy=-1.575491 0.471657 -1.581128 -> xyz=0 0 -0.2 rpy=-1.575491 0.471657 -1.581128
- joint motor_r1: origin xyz=0.5 0 -0.3 rpy=1.57549 0.471558 1.581128 -> xyz=0.25 0 -0.2 rpy=1.57549 0.471558 1.581128
